File: orb/eagle/orb.sch (EAGLE design)
At the start: 22 parts, among them J1 MICRO USB, Q1 CRYSTAL, T1 DMG2302U, T2 DMG2302U, T3 DMG2302U, U1 PRTR5V0U2X, U2 ATTINY2313

Commit message: First iteration of layout. Work in progress.
Parts:
- removed C1: 47U, rcl:CPOL-USCT3216
- removed D1: GREEN, arm-pro-mini:LED
- removed D2: RED, arm-pro-mini:LED
- removed D3: BLUE, arm-pro-mini:LED
- removed U1: PRTR5V0U2X, arm-pro-mini:PRTR5V0U2X
- added C2: 1000U 10V, rcl:CPOL-US153CLV-1010
- added D4: AZ23C3V6, orb:BAS40-06
- added LED1: OVSTRGBBCR4, orb:OVSTRGBBCR4
- added R8: ?? 1W, rcl:R-US_R2512W
- added U$1, U$12, U$2, U$3, U$4, U$5: MOUNTING_HOLE, orb:MOUNTING_HOLE
- Q1: value CRYSTAL -> 12MHZ
- U2: value ATTINY2313 -> ATINY44A; device orb:ATTINY2313-*S* -> orb:TINY24/44/84-SSU
Connections:
- removed net BLUE: T3.G, U2.(OC1B)PB4
- removed net GREEN: T2.G, U2.(AIN0)PB0
- removed net MISO: JP1.1, U2.(MISO)PB6
- removed net MOSI: JP1.4
- removed net N$11: D1.C, R6.2
- removed net N$12: D3.C, R7.2
- removed net RED: T1.G, U2.(OC0A)PB2
- removed net SCK: JP1.3, U2.(UCSK)PB7
- new net MISO/GREEN: JP1.1, T3.G, U2.(PCINT5/OC1B/MISO/DO/ADC5)PA5
- new net MOSI/RED: JP1.4, T2.G, U2.(PCINT6/OC1A/SDA/MOSI/ADC6)PA6
- new net N$8: LED1-R.C, R6.2
- new net N$9: LED1-G.C, R7.2
- new net SCK/BLUE: JP1.3, T1.G, U2.(PCINT4/T1/SCL/USCK/ADC4)PA4
- net +5V: now also C2.+, LED1-B.A, LED1-G.A, LED1-R.A; no longer C1.+, D1.A, D2.A, D3.A, U1.VCC
- net CONN: now also U2.(PCINT2/AIN1/ADC2)PA2; no longer U2.(ICP)PD6
- net DM: now also U2.(PCINT1/AIN0/ADC1)PA1; no longer U2.(INT1)PD3
- net DP: now also U2.(PCINT0/AREF/ADC0)PA0, U2.(PCINT10/INT0/OC0A/CKOUT)PB2; no longer U2.(INT0)PD2
- net GND: now also C2.-, D4.AA, U$1.P$1, U$12.P$1, U$2.P$1, U$3.P$1, U$4.P$1, U$5.P$1; no longer C1.-, U1.GND
- net N$1: now also U2.(PCINT9/XTAL2)PB1; no longer U2.PA1(XTAL2)
- net N$3: now also U2.(PCINT8/XTAL1/CLKI)PB0; no longer U2.PA0(XTAL1)
- net N$4: now also R4.2, R8.1; no longer U2.(MOSI)PB5
- net N$5: now also D4.K1; no longer U1.IO2
- net N$6: now also D4.K2; no longer U1.IO1
- net N$7: now also LED1-B.C, R8.2; no longer D2.C, R4.2
- net RESET: now also U2.(PCINT11/RESET/DW)PB3; no longer U2.PA2(/RESET)
Other:
- note removed: "TODO: add large bypass cap"
- moved on the sheet: C3, C4, C5, J1, JP1, Q1, R1, R2, R3, R4, R5, R6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
