File: cutoff/eagle/cutoff.brd (EAGLE design)
At the start: 40 x 45 mm, 31 parts, among them K1 RELAY, U1 LM2931ADT-5.0RKG, U2 NUD3160, U3 ATMEGA328, Y1 16MHz

Commit message: Completed BOM. Generated library from schematic file.
Parts:
- C1: device beeper:UD-6,3X5,8_NICHICON -> cutoff:UD-6,3X5,8_NICHICON
- C2, C3, C5, C6, C7, C8: device resistor:C0603K -> cutoff:C0603K
- C4: device beeper:A/3216-18R -> cutoff:A/3216-18R
- D3: device ir-control:LED -> cutoff:LED
- R1, R2, R3, R4, R6: device resistor:R0402 -> cutoff:R0402
- R5: value 3K3 -> 1K; device resistor:R0402 -> cutoff:R0402
Changed lines of the file:
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@@
 </autorouter>
 <elements>
-<element name="C1" library="beeper" package="UD-6,3X5,8_NICHICON" value="22uF 40V" x="5.715" y="25.4" smashed="yes">
+<element name="C1" library="cutoff" package="UD-6,3X5,8_NICHICON" value="22uF 40V" x="5.715" y="25.4" smashed="yes">
 <attribute name="NAME" x="5.08" y="29.21" size="1.016" layer="25" font="vector" ratio="10"/>
 <attribute name="VALUE" x="2.54" y="20.955" size="1.016" layer="27"/>
 </element>
-<element name="C5" library="resistor" package="C0603K" value="0.1uF" x="14.464" y="18.364" smashed="yes" rot="R270">
+<element name="C5" library="cutoff" package="C0603K" value="0.1uF" x="14.464" y="18.364" smashed="yes" rot="R270">
 <attribute name="NAME" x="13.602" y="15.749" size="1.016" layer="25" font="vector" ratio="10"/>
 <attribute name="VALUE" x="12.814" y="19.164" size="1.016" layer="27" rot="R270"/>
 </element>
-<element name="C2" library="resistor" package="C0603K" value="0.1uF" x="7.13" y="11.11" smashed="yes" rot="R180">
+<element name="C2" library="cutoff" package="C0603K" value="0.1uF" x="7.13" y="11.11" smashed="yes" rot="R180">
 <attribute name="NAME" x="8.707" y="10.495" size="1.016" layer="25" font="vector" ratio="10"/>
 <attribute name="VALUE" x="7.93" y="12.76" size="1.016" layer="27" rot="R180"/>
 </element>
-<element name="C6" library="resistor" package="C0603K" value="0.1uF" x="22.733" y="4.699" smashed="yes" rot="R180">
+<element name="C6" library="cutoff" package="C0603K" value="0.1uF" x="22.733" y="4.699" smashed="yes" rot="R180">
 <attribute name="NAME" x="19.393" y="5.222" size="1.016" layer="25" font="vector" ratio="10"/>
 <attribute name="VALUE" x="23.533" y="6.349" size="1.016" layer="27" rot="R180"/>
 </element>
-<element name="C4" library="beeper" package="A/3216-18R" value="10uF" x="16.435" y="19.275" smashed="yes" rot="R90">
+<element name="C4" library="cutoff" package="A/3216-18R" value="10uF" x="16.435" y="19.275" smashed="yes" rot="R90">
 <attribute name="NAME" x="17.706" y="18.855" size="1.016" layer="25" font="vector" ratio="10"/>
 <attribute name="VALUE" x="18.76" y="17.325" size="1.27" layer="27" rot="R90"/>
 </element>
-<element name="C3" library="resistor" package="C0603K" value="0.1uF" x="3.81" y="6.35" smashed="yes" rot="R90">
+<element name="C3" library="cutoff" package="C0603K" value="0.1uF" x="3.81" y="6.35" smashed="yes" rot="R90">
 <attribute name="NAME" x="3.01" y="8.27" size="1.016" layer="25" font="vector" ratio="10"/>
 <attribute name="VALUE" x="5.46" y="5.55" size="1.016" layer="27" rot="R90"/>
@@
 <attribute name="VALUE" x="31.83" y="10.08" size="1.27" layer="27" rot="R270"/>
 </element>
-<element name="R1" library="resistor" package="R0402" value="10K" x="6.35" y="6.35" smashed="yes" rot="R270">
+<element name="R1" library="cutoff" package="R0402" value="10K" x="6.35" y="6.35" smashed="yes" rot="R270">
 <attribute name="NAME" x="5.715" y="8.255" size="1.016" layer="25" font="vector" ratio="10"/>
 <attribute name="VALUE" x="4.445" y="6.985" size="1.27" layer="27" rot="R270"/>
 </element>
-<element name="R2" library="resistor" package="R0402" value="10K" x="8.89" y="6.35" smashed="yes" rot="R270">
+<element name="R2" library="cutoff" package="R0402" value="10K" x="8.89" y="6.35" smashed="yes" rot="R270">
 <attribute name="NAME" x="8.255" y="8.255" size="1.016" layer="25" font="vector" ratio="10"/>
 <attribute name="VALUE" x="6.985" y="6.985" size="1.27" layer="27" rot="R270"/>
 </element>
-<element name="R5" library="resistor" package="R0402" value="3K3" x="33.57" y="20.805" smashed="yes" rot="R270">
+<element name="R5" library="cutoff" package="R0402" value="1K" x="33.57" y="20.805" smashed="yes" rot="R270">
 <attribute name="NAME" x="35.518" y="20.089" size="1.016" layer="25" font="vector" ratio="10" rot="R90"/>
 <attribute name="VALUE" x="31.665" y="21.44" size="1.27" layer="27" rot="R270"/>
 </element>
-<element name="R6" library="resistor" package="R0402" value="10K" x="16.75" y="12.51" smashed="yes" rot="R90">
+<element name="R6" library="cutoff" package="R0402" value="10K" x="16.75" y="12.51" smashed="yes" rot="R90">
 <attribute name="NAME" x="15.861" y="12.002" size="1.016" layer="25" font="vector" ratio="10" rot="R90"/>
 <attribute name="VALUE" x="18.655" y="11.875" size="1.27" layer="27" rot="R90"/>
@@
 <attribute name="VALUE" x="30.845" y="29.21" size="1.27" layer="27" rot="R90"/>
 </element>
-<element name="R3" library="resistor" package="R0402" value="60K" x="13.335" y="24.765" smashed="yes" rot="R90">
+<element name="R3" library="cutoff" package="R0402" value="60K" x="13.335" y="24.765" smashed="yes" rot="R90">
 <attribute name="NAME" x="12.446" y="24.13" size="1.016" layer="25" font="vector" ratio="10" rot="R90"/>
 <attribute name="VALUE" x="15.24" y="24.13" size="1.27" layer="27" rot="R90"/>
 </element>
-<element name="R4" library="resistor" package="R0402" value="30K" x="15.875" y="24.765" smashed="yes" rot="R270">
+<element name="R4" library="cutoff" package="R0402" value="30K" x="15.875" y="24.765" smashed="yes" rot="R270">
 <attribute name="NAME" x="17.78" y="24.13" size="1.016" layer="25" font="vector" ratio="10" rot="R90"/>
 <attribute name="VALUE" x="13.97" y="25.4" size="1.27" layer="27" rot="R270"/>
@@
 <attribute name="VALUE" x="9.365" y="21.905" size="1.27" layer="27" rot="R180"/>
 </element>
-<element name="D3" library="ir-control" package="LED" value="LED" x="29.21" y="24.13" smashed="yes" rot="R90">
+<element name="D3" library="cutoff" package="LED" value="LED" x="29.21" y="24.13" smashed="yes" rot="R90">
 <attribute name="NAME" x="31.623" y="23.495" size="1.016" layer="25" font="vector" ratio="10"/>
 <attribute name="VALUE" x="33.528" y="22.86" size="1.27" layer="27" ratio="10" rot="R90"/>
@@
 <attribute name="VALUE" x="13.295" y="28.48" size="1.27" layer="27" rot="R90"/>
 </element>
-<element name="C7" library="resistor" package="C0603K" value="0.1uF" x="27.05" y="18.965" smashed="yes" rot="R90">
+<element name="C7" library="cutoff" package="C0603K" value="0.1uF" x="27.05" y="18.965" smashed="yes" rot="R90">
 <attribute name="NAME" x="27.86" y="18.429" size="1.016" layer="25" font="vector" ratio="10"/>
 <attribute name="VALUE" x="28.7" y="18.165" size="1.016" layer="27" rot="R90"/>
 </element>
-<element name="C8" library="resistor" package="C0603K" value="0.1uF" x="25" y="19" smashed="yes" rot="R90">
+<element name="C8" library="cutoff" package="C0603K" value="0.1uF" x="25" y="19" smashed="yes" rot="R90">
 <attribute name="NAME" x="24.121" y="20.825" size="1.016" layer="25" font="vector" ratio="10"/>
 <attribute name="VALUE" x="26.65" y="18.2" size="1.016" layer="27" rot="R90"/>
