File: battery_cutoff/eagle/cutoff.brd (EAGLE design)
At the start: 40 x 45 mm, 31 parts, among them K1 RELAY, U1 LM2931ADT-5.0RKG, U2 NUD3160, U3 ATMEGA328, Y1 16MHz

Commit message: Updated files for actual V1 built.
Parts:
- R5: value 1K -> 330
Changed lines of the file:
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@@
 <attribute name="VALUE" x="6.985" y="6.985" size="1.27" layer="27" rot="R270"/>
 </element>
-<element name="R5" library="cutoff" package="R0402" value="1K" x="33.57" y="20.805" smashed="yes" rot="R270">
+<element name="R5" library="cutoff" package="R0402" value="330" x="33.57" y="20.805" smashed="yes" rot="R270">
 <attribute name="NAME" x="35.518" y="20.089" size="1.016" layer="25" font="vector" ratio="10" rot="R90"/>
 <attribute name="VALUE" x="31.665" y="21.44" size="1.27" layer="27" rot="R270"/>
