File: battery_cutoff/eagle/cutoff.sch (EAGLE design)
At the start: 31 parts, among them K1 RELAY, U1 LM2931ADT-5.0RKG, U2 NUD3160, U3 ATMEGA328, Y1 16MHz

Commit message: Updated files for actual V1 built.
Parts:
- R5: value 1K -> 330
Changed lines of the file:
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@@
 </classes>
 <parts>
-<part name="R5" library="cutoff" deviceset="R-US_" device="R0402" value="1K"/>
+<part name="R5" library="cutoff" deviceset="R-US_" device="R0402" value="330"/>
 <part name="GND6" library="cutoff" deviceset="GND" device=""/>
 <part name="C2" library="cutoff" deviceset="C-US" device="C0603K" value="0.1uF"/>
