File: soap_dispenser/kicad/soap_dispenser.sch (KiCad schematic (older format))
At the start: 33 parts, among them M1 Motor_DC, Q1 PMOS, Q11 NMOS, Q3 PMOS, Q4 NMOS, Q5 NMOS, SW1 SW_SPDT, SW8 SW_Push, U1 ATtiny48-AU

Commit message: Minor schema tweaks.
Parts:
- removed D4: LED_Dual_CAC, symbol Device:LED_Dual_CAC
- added D4A: RED, symbol Device:LED
- added D4B: YELLOW, symbol Device:LED
- added R15, R16: 10K, symbol Device:R_Small_US
- added TP19: TestPoint, symbol Connector:TestPoint
Connections:
- net OPEN is gone; now on net #DOOR_CLOSED: J?.3 (Pin_3)
- net +3V6: now also D4A.2 (A), D4B.2 (A)
- net GNDD: now also R15.1, R16.1, TP19.1
- net X1: now also Q5.2 (G), U1.32 (PD2), R16.2; no longer R6.1, U1.31 (PD1)
- net X2: now also R6.1, U1.31 (PD1); no longer Q5.2 (G), U1.32 (PD2)
- net Y1: now also Q4.2 (G), TP3.1, U1.1 (PD3), R15.2; no longer R10.1, TP8.1, U1.8 (PB7)
- net Y2: now also R10.1, TP8.1, U1.8 (PB7); no longer Q4.2 (G), TP3.1, U1.1 (PD3)
- net at RN5B.2, TP20.1: now also D4B.1 (K)
- net at RN5A.2, TP21.1: now also D4A.1 (K)
Other:
- note removed: "LOGIC 1"
- note removed: "LOGIC 2"
- note removed: "LOGIC 3\n"
- note removed: "LOGIC 4\n"
- note removed: "LOGIC 5\n"
- note removed: "LOGIC 6\n"
- moved on the sheet: C?, RN5A, RN5B, RN6B?, TP20, TP21

Commit message: Deleted kicad backup files.
Other:
- note added: "Forward"
- note added: "Idle"
- note added: "MODE"
- note added: "Reverse"
- note added: "Stop Forward"
- note added: "Stop Reverse"
- note added: "X"
- note added: "X1"
- note added: "X2"
- note added: "Y1"
- note added: "Y2"
Changed lines of the file:
@@
 Wire Wire Line
 	5550 4300 5550 4500
+Text Notes 4000 6600 0    50   ~ 0
+Idle
+Text Notes 4000 6700 0    50   ~ 0
+Forward
+Text Notes 4000 6800 0    50   ~ 0
+Stop Forward
+Text Notes 4000 6900 0    50   ~ 0
+Reverse
+Text Notes 4000 7000 0    50   ~ 0
+Stop Reverse
+Wire Notes Line
+	4600 6400 4600 7000
+Wire Notes Line
+	4800 6400 4800 7000
+Wire Notes Line
+	5000 6400 5000 7000
+Wire Notes Line
+	5200 6400 5200 7000
+Wire Notes Line
+	5400 6400 5400 7000
+Text Notes 4650 6500 0    50   ~ 0
+Y2
+Text Notes 4850 6500 0    50   ~ 0
+Y1
+Text Notes 5050 6500 0    50   ~ 0
+X2
+Text Notes 5250 6500 0    50   ~ 0
+X1
+Text Notes 4650 6700 0    50   ~ 0
+X
+Text Notes 5250 6700 0    50   ~ 0
+X
+Wire Notes Line
+	3900 6400 3900 7000
+Wire Notes Line
+	3900 7000 5400 7000
+Wire Notes Line
+	3900 6900 5400 6900
+Wire Notes Line
+	3900 6800 5400 6800
+Wire Notes Line
+	3900 6700 5400 6700
+Wire Notes Line
+	3900 6600 5400 6600
+Wire Notes Line
+	3900 6500 5400 6500
+Text Notes 4000 6500 0    50   ~ 0
+MODE
+Wire Notes Line
+	3900 6400 5400 6400
 $EndSCHEMATC

Commit message: Work in progress
Parts:
- added Q?: NMOS, symbol Device:Q_NMOS_DGS
- added R19: 0R15, symbol Device:R_Small_US
- added R23: 120K, symbol Device:R_Small_US
- added R26: 10K, symbol Device:R_Small_US
- added R?: 1M, symbol Device:R_Small_US
- added TP6: TestPoint, symbol Connector:TestPoint
Connections:
- net +3V6: now also R?.2
- net GNDD: now also Q?.3 (S), R19.1; no longer Q4.3 (S), Q5.3 (S)
- net CURRENT1: now reaches U1.10 (PD6)
- net CURRENT1: now also R23.1
- net CURRENT2: now reaches U1.27 (PC4)
- net CURRENT2: now also Q?.1 (D), R?.1, TP6.1
- net #ACTIVE renamed PARKING
- net #DOOR_CLOSED renamed DOOR_OPENED
- new net: Q4.3 (S), Q5.3 (S), R19.2, R26.2
- new net: Q?.2 (G), R23.2, R26.1
Other:
- moved on the sheet: C?, D4A, D4B, R9, RN5A, RN5B, RN6B?, TP19, TP2, TP20, TP21
