File: stepper_analyzer/kicad/main/stepper_analyzer.sch (KiCad schematic (older format))
At the start: 36 parts, among them J1 Conn_01x04, J2 Conn_01x04, M1 Stepper_Motor_bipolar, SW1 SW_Push, SW2 SW_Push, U1 ACS70331, U2 ACS70331, U3 Teensy4, U4 TFT

Commit message: Work in progress.
Parts:
- added SW3: SW_DIP_x04, stepper_analyzer:SW_DIP_SPSTx04_Slide_Copal_CHS-04B_W7.62mm_P1.27mm, symbol stepper_analyzer:SW_DIP_x04
- M1: footprint (none) -> stepper_analyzer:NO_PADS
- R1, R2, R3, R4, R5: footprint stepper_analyzer:R_0201_0603Metric -> stepper_analyzer:R_0603_1608Metric
- U1, U2: value ACS70331 -> ACS70331EESATR-2P5U3
- U3: value Teensy4 -> Teensy 4,0; symbol stepper_analyzer:Teensy4 -> stepper_analyzer-rescue:Teensy4-stepper_analyzer
- renumbered GND to GND1
Connections:
- wire segments 120 -> 133
Other:
- note added: "+/- 2.5A"
- note added: "1.8" 128x160 pixels, color TFT\nSPI, ST7735 controller"
- note added: "CONFIGURATION"
- note added: "OUT"
- note added: "Optional, for firmware developement."
- note added: "To Stepper\nController"
- note removed: "TODO: swap ADC1, ADC2 inputs ?"
- moved on the sheet: D1, D2, D3, GND1, J1, J2, R1, R2, R3, RV1, RV2, TP1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

Commit message: Work in progress.
Parts:
- removed M1: Stepper_Motor_bipolar, stepper_analyzer:NO_PADS, symbol stepper_analyzer:Stepper_Motor_bipolar
- added R6: 400R, stepper_analyzer:R_0603_1608Metric, symbol Device:R_Small_US
Connections:
- net +3V3: now also R6.1; no longer RV1.3, RV2.3
- net ~A: now reaches J1.1 (Pin_1), J2.1 (Pin_1)
- net ~B: now reaches J1.4 (Pin_4), J2.4 (Pin_4)
- net A: now reaches J1.2 (Pin_2), U2.2 (-)
- net B: now reaches J1.3 (Pin_3), U1.2 (-)
- new net: R6.2, RV1.3, RV2.3
Other:
- note added: "+/-2,5A\n"
- note added: "1.5V + 0.4xI1"
- note added: "3VDC"
- note added: "A"
- note added: "B"
- note added: "CONFIGURATION\nSWITCHES"
- note added: "Connectors J1, J2 are\ninterchangeable"
- note added: "I1\n"
- note added: "I2\n"
- note added: "LEFT\nBUTTON"
- note added: "RIGHT\nBUTTON"
- note added: "SMD 1.27mm pitch\n"
- note removed: "+/- 2.5A"
- note removed: "CONFIGURATION"
- note removed: "IN"
- note removed: "OUT"
Changed lines of the file:
@@
-$EndComp
-$Comp
-L stepper_analyzer:3V3 #PWR01
-U 1 1 5DB2A2D4
-P 1700 6750
-F 0 "#PWR01" H 1700 6600 50  0001 C CNN
-F 1 "3V3" H 1715 6923 50  0000 C CNN
-F 2 "" H 1700 6750 50  0001 C CNN
-F 3 "" H 1700 6750 50  0001 C CNN
-	1    1700 6750
-	1    0    0    -1
 $EndComp
 $Comp
 L stepper_analyzer:3V3 #PWR03
 U 1 1 5DB2AA08
-P 2600 6750
-F 0 "#PWR03" H 2600 6600 50  0001 C CNN
-F 1 "3V3" H 2615 6923 50  0000 C CNN
-F 2 "" H 2600 6750 50  0001 C CNN
-F 3 "" H 2600 6750 50  0001 C CNN
-	1    2600 6750
+P 2150 6300
+F 0 "#PWR03" H 2150 6150 50  0001 C CNN
+F 1 "3V3" H 2165 6473 50  0000 C CNN
+F 2 "" H 2150 6300 50  0001 C CNN
+F 3 "" H 2150 6300 50  0001 C CNN
+	1    2150 6300
 	1    0    0    -1
 $EndComp
@@
 Wire Wire Line
 	2850 6950 2750 6950
-Text Notes 1800 1650 0    50   ~ 0
-IN
-Text Notes 2700 1650 0    50   ~ 0
-OUT
 Wire Wire Line
 	4650 5250 4650 5300
@@
 Wire Wire Line
 	1700 7100 1700 7150
-Wire Wire Line
-	1700 6750 1700 6800
-Wire Wire Line
-	2600 6750 2600 6800
 Wire Wire Line
 	3550 6450 3600 6450
@@
 Wire Wire Line
 	5050 2500 4950 2500
-$Comp
-L stepper_analyzer:Stepper_Motor_bipolar M1
-U 1 1 5DC305A6
-P 2300 1300
-F 0 "M1" H 2528 1365 50  0001 L CNN
-F 1 "Stepper_Motor_bipolar" H 2488 1333 50  0001 L CNN
-F 2 "stepper_analyzer:NO_PADS" H 2310 1290 50  0001 C CNN
-F 3 "" H 2310 1290 50  0001 C CNN
-	1    2300 1300
-	1    0    0    -1
-$EndComp
 $Comp
 L stepper_analyzer:3V3 #PWR0101
@@
 U 1 1 5DAA891F
 P 3900 2600
-F 0 "U2" H 3400 3250 50  0000 C CNN
-F 1 "ACS70331EESATR-2P5U3" H 3300 3100 50  0000 C CNN
+F 0 "U2" H 3350 3150 50  0000 C CNN
+F 1 "ACS70331EESATR-2P5U3" H 3250 3000 50  0000 C CNN
 F 2 "Sensor_Current:Allegro_QFN-12-10-1EP_3x3mm_P0.5mm" H 4300 2550 50  0001 L CIN
 F 3 "" H 3900 2600 50  0001 C CNN
@@
 	2300 2100 2300 1800
 Wire Wire Line
-	1700 1800 1700 1950
-Wire Wire Line
-	1700 1950 2600 1950
-Wire Wire Line
-	2600 1950 2600 1800
+	1700 1800 1700 2000
+Wire Wire Line
+	1700 2000 2600 2000
+Wire Wire Line
+	2600 2000 2600 1800
 Wire Wire Line
 	1600 1800 1600 4050
@@
 	2400 1800 2400 2450
 Wire Wire Line
-	2500 1800 2500 2250
-Wire Wire Line
-	2500 2250 1900 2250
-Wire Wire Line
-	1900 2250 1900 3750
-Text Notes 1850 4500 0    50   ~ 0
-+/- 2.5A
-Text Notes 3200 2250 0    50   ~ 0
-+/- 2.5A
+	2500 1800 2500 2200
+Wire Wire Line
+	2500 2200 1900 2200
+Wire Wire Line
+	1900 2200 1900 3750
+Text Notes 2750 2400 0    50   ~ 0
+I2\n
 Wire Wire Line
 	6600 2050 6600 2000
@@
 P 6800 2350
 F 0 "SW3" V 6950 2900 50  0000 R CNN
-F 1 "SW_DIP_x04" V 6800 3150 50  0000 R CNN
+F 1 "SW_DIP_x04" V 6800 3150 50  0001 R CNN
 F 2 "stepper_analyzer:SW_DIP_SPSTx04_Slide_Copal_CHS-04B_W7.62mm_P1.27mm" H 6800 2350 50  0001 C CNN
 F 3 "~" H 6800 2350 50  0001 C CNN
@@
 Wire Wire Line
 	6900 2650 6900 2750
-Text Notes 6450 1900 0    50   ~ 0
-CONFIGURATION
-Text Notes 1400 1350 0    50   ~ 0
+Text Notes 6500 1900 0    50   ~ 0
+CONFIGURATION\nSWITCHES
+Text Notes 1350 1450 0    50   ~ 0
 To Stepper\nController
+$Comp
+L Device:R_Small_US R6
+U 1 1 5DB2651A
+P 2150 6450
+F 0 "R6" H 1950 6550 50  0000 C CNN
+F 1 "400R" H 1950 6450 50  0000 C CNN
+F 2 "stepper_analyzer:R_0603_1608Metric" H 2150 6450 50  0001 C CNN
+F 3 "~" H 2150 6450 50  0001 C CNN
+	1    2150 6450
+	1    0    0    -1
+$EndComp
+Wire Wire Line
+	1700 6650 2150 6650
+Wire Wire Line
+	1700 6650 1700 6800
+Wire Wire Line
+	2600 6650 2600 6800
+Wire Wire Line
+	2150 6550 2150 6650
+Wire Wire Line
+	2150 6350 2150 6300
+Connection ~ 2150 6650
+Wire Wire Line
+	2150 6650 2600 6650
+Text Notes 2350 6600 0    50   ~ 0
+3VDC
+Text Notes 2850 1300 0    50   ~ 0
+Connectors J1, J2 are\ninterchangeable
+Text Notes 4850 2850 0    50   ~ 0
+1.5V + 0.4xI1
+Text Notes 4350 4200 0    50   ~ 0
+1.5V + 0.4xI1
+Text Notes 2650 2550 0    50   ~ 0
++/-2,5A\n
+Text Notes 1950 3050 0    50   ~ 0
+I1\n
+Text Notes 1950 3150 0    50   ~ 0
++/-2,5A\n
+Text Notes 5700 2350 0    50   ~ 0
+SMD 1.27mm pitch\n
+Text Notes 5800 5750 0    50   ~ 0
+RIGHT\nBUTTON
+Text Notes 5350 5750 0    50   ~ 0
+LEFT\nBUTTON
+Text Label 1600 1900 0    50   ~ 0
+B
+Text Label 1700 1900 0    50   ~ 0
+~B
+Text Label 1400 1900 2    50   ~ 0
+~A
+Text Label 1500 1900 2    50   ~ 0
+A
+Text Notes 2325 1475 0    50   ~ 0
+A
+Text Notes 2525 1475 0    50   ~ 0
+B
 $EndSCHEMATC

Commit message: Work in progress
Parts:
- C3, C4: value 0.1uF -> 0.22uF
Connections:
- net +3V3 renamed +3V3A
- net +3V3A: no longer C5.1, U3.16 (3V3_OUT), U4.2 (3V3)
- new net +3V3D: C5.1, U3.16 (3V3_OUT), U4.2 (3V3)
- no-connect marks 0 -> 1
Other:
- note added: "+/- 2.5A isolated current sensor\nVout = 1.5V +/- 0.4V per Amp.\n"
- note added: "I2"
- note added: "Resistors, capacitors and LEDS are 0603 SMD packages."
- note added: "TODO: add stepper motor symbol after completing the pcb layout"
- note removed: "+/-2,5A\n"
- note removed: "1.5V + 0.4xI1"
- note removed: "I2\n"
- moved on the sheet: D1, D2, D3, GND1, R1, R2, R3, R6, RV1, RV2, TP1, TP2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

Commit message: Sent PCB to fabrication.
Parts:
- added M?: Stepper_Motor_bipolar, symbol stepper_analyzer:Stepper_Motor_bipolar
Changed lines of the file:
@@
 Wire Notes Line
 	1200 7550 5275 7550
+$Comp
+L stepper_analyzer:Stepper_Motor_bipolar M?
+U 1 1 5DB96B5F
+P 2300 1325
+F 0 "M?" H 2350 1725 50  0001 L CNN
+F 1 "Stepper_Motor_bipolar" H 2200 1675 50  0001 L TNN
+F 2 "" H 2310 1415 50  0001 C CNN
+F 3 "http://www.infineon.com/dgdl/Application-Note-TLE8110EE_driving_UniPolarStepperMotor_V1.1.pdf?fileId=db3a30431be39b97011be5d0aa0a00b0" H 2310 1415 50  0001 C CNN
+	1    2300 1325
+	1    0    0    -1
+$EndComp
 $EndSCHEMATC

Commit message: Work in progress
Parts:
- U1, U2: value ACS70331EESATR-2P5U3 -> ACS70331EESATR-2P5B3
Changed lines of the file:
@@
 P 3900 2600
 F 0 "U2" H 3350 3150 50  0000 C CNN
-F 1 "ACS70331EESATR-2P5U3" H 3250 3000 50  0000 C CNN
+F 1 "ACS70331EESATR-2P5B3" H 3250 3000 50  0000 C CNN
 F 2 "Sensor_Current:Allegro_QFN-12-10-1EP_3x3mm_P0.5mm" H 4300 2550 50  0001 L CIN
 F 3 "" H 3900 2600 50  0001 C CNN
@@
 P 2700 3900
 F 0 "U1" H 2050 3600 50  0000 C CNN
-F 1 "ACS70331EESATR-2P5U3" H 2050 3275 50  0000 C CNN
+F 1 "ACS70331EESATR-2P5B3" H 2050 3275 50  0000 C CNN
 F 2 "Sensor_Current:Allegro_QFN-12-10-1EP_3x3mm_P0.5mm" H 3100 3850 50  0001 L CIN
 F 3 "" H 2700 3900 50  0001 C CNN
