File: stepper_analyzer/kicad/main/stepper_analyzer.sch (KiCad schematic (older format))
At the start: 32 parts, among them J1 Conn_01x04, J2 Conn_01x04, J3 Conn_01x05, J4 Conn_01x04_Female, M1 Stepper_Motor_bipolar, U1 ACS70331, U2 ACS70331, U3 Teensy4-stepper_analyzer

Commit message: Generated gerbers.
Parts:
- C1, C2, C3, C4: value C_Small -> 100nf
- R1, R2, R3: value R_Small_US -> 3K3
- R4, R5: value R_Small_US -> 330R
Connections:
- no-connect marks 2 -> 3
Other:
- note added: "For development only\n"
Changed lines of the file:
@@
 P 4050 2050
 F 0 "C2" V 3821 2050 50  0000 C CNN
-F 1 "C_Small" V 3912 2050 50  0000 C CNN
+F 1 "100nf" V 3912 2050 50  0000 C CNN
 F 2 "stepper_analyzer:C_0603_1608Metric" H 4050 2050 50  0001 C CNN
 F 3 "~" H 4050 2050 50  0001 C CNN
@@
 P 2850 3350
 F 0 "C1" V 2621 3350 50  0000 C CNN
-F 1 "C_Small" V 2712 3350 50  0000 C CNN
+F 1 "100nf" V 2712 3350 50  0000 C CNN
 F 2 "stepper_analyzer:C_0603_1608Metric" H 2850 3350 50  0001 C CNN
 F 3 "~" H 2850 3350 50  0001 C CNN
@@
 P 5550 3100
 F 0 "R5" V 5345 3100 50  0000 C CNN
-F 1 "R_Small_US" V 5436 3100 50  0000 C CNN
+F 1 "330R" V 5436 3100 50  0000 C CNN
 F 2 "stepper_analyzer:R_0603_1608Metric" H 5550 3100 50  0001 C CNN
 F 3 "~" H 5550 3100 50  0001 C CNN
@@
 P 3475 6650
 F 0 "R1" H 3375 6700 50  0000 C CNN
-F 1 "R_Small_US" H 3375 6600 50  0000 C CNN
+F 1 "3K3" H 3375 6600 50  0000 C CNN
 F 2 "stepper_analyzer:R_0603_1608Metric" H 3475 6650 50  0001 C CNN
 F 3 "~" H 3475 6650 50  0001 C CNN
@@
 P 3875 6650
 F 0 "R2" H 3775 6700 50  0000 C CNN
-F 1 "R_Small_US" H 3775 6600 50  0000 C CNN
+F 1 "3K3" H 3775 6600 50  0000 C CNN
 F 2 "stepper_analyzer:R_0603_1608Metric" H 3875 6650 50  0001 C CNN
 F 3 "~" H 3875 6650 50  0001 C CNN
@@
 P 4275 6650
 F 0 "R3" H 4175 6700 50  0000 C CNN
-F 1 "R_Small_US" H 4175 6600 50  0000 C CNN
+F 1 "3K3" H 4175 6600 50  0000 C CNN
 F 2 "stepper_analyzer:R_0603_1608Metric" H 4275 6650 50  0001 C CNN
 F 3 "~" H 4275 6650 50  0001 C CNN
@@
 P 5750 3250
 F 0 "C4" H 5950 3300 50  0000 C CNN
-F 1 "C_Small" H 5925 3400 50  0000 C CNN
+F 1 "100nf" H 5925 3400 50  0000 C CNN
 F 2 "stepper_analyzer:C_0603_1608Metric" H 5750 3250 50  0001 C CNN
 F 3 "~" H 5750 3250 50  0001 C CNN
@@
 U 1 1 5DAAD3D8
 P 3900 3800
-F 0 "JP1" H 3900 4004 50  0000 C CNN
-F 1 "Jumper_3_Bridged12" H 3700 3925 50  0000 C CNN
+F 0 "JP1" H 3925 3925 50  0000 C CNN
+F 1 "Jumper_3_Bridged12" H 3700 3925 50  0001 C CNN
 F 2 "stepper_analyzer:PinHeader_1x03_P2.54mm_Vertical" H 3900 3800 50  0001 C CNN
 F 3 "~" H 3900 3800 50  0001 C CNN
@@
 P 5050 4050
 F 0 "R4" V 4845 4050 50  0000 C CNN
-F 1 "R_Small_US" V 4936 4050 50  0000 C CNN
+F 1 "330R" V 4936 4050 50  0000 C CNN
 F 2 "stepper_analyzer:R_0603_1608Metric" H 5050 4050 50  0001 C CNN
 F 3 "~" H 5050 4050 50  0001 C CNN
@@
 P 5250 4200
 F 0 "C3" H 5075 4200 50  0000 C CNN
-F 1 "C_Small" H 5000 4300 50  0000 C CNN
+F 1 "100nf" H 5000 4300 50  0000 C CNN
 F 2 "stepper_analyzer:C_0603_1608Metric" H 5250 4200 50  0001 C CNN
 F 3 "~" H 5250 4200 50  0001 C CNN
@@
 POT2
 NoConn ~ 7500 3150
+NoConn ~ 8500 3600
+Text Notes 2425 6000 0    50   ~ 0
+For development only\n
 $EndSCHEMATC

Commit message: Version 1.1
Parts:
- U3: value Teensy4-stepper_analyzer -> Teensy4
Other:
- note added: "+/- 2.5A isolated current sensors\nVout = 1.5V +/- 0.4V per Amp.\n"
- note added: "Connectors J1, J2 are interchangeable.\nEach can be used as input or output."
- note removed: "+/- 2.5A isolated current sensor\nVout = 1.5V +/- 0.4V per Amp.\n"
- note removed: "Connectors J1, J2 are\ninterchangeable"
- note removed: "SMD 1.27mm pitch\n"
- note removed: "TODO: add stepper motor symbol after completing the pcb layout"
- note removed: "TODO: check footprints sizes"
- note removed: "TODO: check netlist"
Changed lines of the file:
@@
 P 6800 4200
 F 0 "U3" H 7250 3200 50  0000 C CNN
-F 1 "Teensy4-stepper_analyzer" H 7300 3100 50  0000 C CNN
+F 1 "Teensy4" H 7300 3100 50  0000 C CNN
 F 2 "stepper_analyzer:TEENSY40" H 6750 4200 50  0001 C CIN
 F 3 "" H 6750 4200 50  0001 C CNN
@@
 Text Notes 4450 700  0    50   ~ 0
 TODO: Verify pin numbers
-Text Notes 4450 875  0    50   ~ 0
-TODO: check footprints sizes
 Connection ~ 2650 3350
 $Comp
@@
 	5250 4050 6100 4050
 Connection ~ 5250 4050
-Text Notes 4450 1050 0    50   ~ 0
-TODO: check netlist
 Wire Wire Line
 	2100 3750 1900 3750
@@
 Text Notes 1350 1450 0    50   ~ 0
 To Stepper\nController
-Text Notes 2850 1300 0    50   ~ 0
-Connectors J1, J2 are\ninterchangeable
+Text Notes 1300 875  0    50   ~ 0
+Connectors J1, J2 are interchangeable.\nEach can be used as input or output.
 Text Notes 3125 2425 0    50   ~ 0
 I2
 Text Notes 1975 3725 0    50   ~ 0
 I1\n
-Text Notes 5800 2550 0    50   ~ 0
-SMD 1.27mm pitch\n
 Text Label 1600 1900 0    50   ~ 0
 B
@@
 Text Notes 2525 1475 0    50   ~ 0
 B
-Text Notes 4450 1225 0    50   ~ 0
-TODO: add stepper motor symbol after completing the pcb layout
 NoConn ~ 7500 4150
 Text Notes 6275 6550 0    50   ~ 0
@@
 	0    1    1    0
 $EndComp
-Text Notes 1575 5000 0    50   ~ 0
-+/- 2.5A isolated current sensor\nVout = 1.5V +/- 0.4V per Amp.\n
+Text Notes 3275 4450 0    50   ~ 0
++/- 2.5A isolated current sensors\nVout = 1.5V +/- 0.4V per Amp.\n
 $Comp
 L stepper_analyzer:Stepper_Motor_bipolar M1
