File: stepper_analyzer/kicad/main/stepper_analyzer.kicad_pcb (KiCad board)
At the start: 2 copper layers, 81.3 x 66 mm, 35 parts, among them J1 Conn_01x04, J2 Conn_01x04, SW1 SW_Push, SW2 SW_Push, U1 ACS70331, U2 ACS70331, U3 Teensy4, U4 TFT

Commit message: Work in progress.
Parts:
- removed the TP1 at (139.3, 78.1)
- added CH2: TestPoint, stepper_analyzer:TestPoint_Loop_D1.80mm_Drill1.0mm_Beaded, F.Cu at (137.2, 76.2)
- added M1: Stepper_Motor_bipolar, stepper_analyzer:NO_PADS, F.Cu at (154.0, 32.6)
- added SW3: SW_DIP_x04, stepper_analyzer:SW_DIP_SPSTx04_Slide_Copal_CHS-04B_W7.62mm_P1.27mm, F.Cu at (134.9, 108.0)
- R1, R2, R3, R4, R5: footprint stepper_analyzer:R_0201_0603Metric -> stepper_analyzer:R_0603_1608Metric
- U1, U2: value ACS70331 -> ACS70331EESATR-2P5U3
- U3: value Teensy4 -> Teensy 4,0
- moved C3 16.2 mm to (118.8, 80.6), turned to 0 degrees
- moved R5 14.5 mm to (137.6, 80.6), turned to 0 degrees
- moved C4 14.2 mm to (134.0, 80.5)
- moved J2 13.0 mm to (134.9, 64.3)
- moved J1 12.7 mm to (122.2, 64.3)
- moved SW2 9.32 mm to (181.4, 125.0), turned to 180 degrees
- moved SW1 8.10 mm to (160.8, 125.0), turned to 180 degrees
- moved R4 7.38 mm to (123.4, 80.6), turned to 0 degrees
- moved R3 6.86 mm to (117.1, 113.8), turned to 0 degrees
- moved R2 5.74 mm to (117.1, 108.7), turned to 0 degrees
- moved R1 5.53 mm to (117.1, 103.6), turned to 0 degrees
- moved C2 2.50 mm to (137.2, 73.4)
- moved U2 2.36 mm to (137.2, 69.8)
- moved CH1 2.07 mm to (124.5, 76.2)
- moved JP2 2.05 mm to (142.2, 71.1)
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- renumbered TP2 to CH1, TP3 to GND1, TP4 to TP1, TP5 to TP2, TP6 to TP3
Connections:
- J2 pad 3: Net-(J1-Pad3) -> Net-(J2-Pad3)
- J2 pad 4: Net-(J2-Pad4) -> Net-(J1-Pad4)
- JP1 pad 3: POT2 -> POT1
- JP2 pad 3: POT1 -> POT2
- U1 pad 1: Net-(J1-Pad2) -> Net-(J2-Pad3)
- U1 pad 2: Net-(J2-Pad2) -> Net-(J1-Pad3)
- U2 pad 1: Net-(J1-Pad4) -> Net-(J2-Pad2)
- U2 pad 2: Net-(J2-Pad4) -> Net-(J1-Pad2)
- U3 pad 24: Net-(C3-Pad2) -> Net-(C4-Pad2)
- U3 pad 30: Net-(C4-Pad2) -> Net-(C3-Pad2)
- U3 pad 6: (no net) -> Net-(SW3-Pad1)
- U3 pad 7: (no net) -> Net-(SW3-Pad2)
- U3 pad 8: (no net) -> Net-(SW3-Pad3)
- U3 pad 9: (no net) -> Net-(SW3-Pad4)

Commit message: Work in progress.
Parts:
- removed M1: Stepper_Motor_bipolar, stepper_analyzer:NO_PADS
- added R6: 400R, stepper_analyzer:R_0603_1608Metric, F.Cu at (124.2, 109.5)
- moved D1 10.9 mm to (118.1, 116.3)
- moved TP1 10.9 mm to (114.3, 116.3)
- moved R1 10.7 mm to (118.1, 114.3)
- moved R3 9.71 mm to (118.1, 104.1)
- moved D3 9.40 mm to (118.1, 106.2)
- moved TP3 9.40 mm to (114.3, 106.2)
- moved R4 2.25 mm to (121.9, 82.3)
- moved CH2 2.22 mm to (136.7, 78.4)
- moved CH1 2.22 mm to (124.0, 78.4)
- moved C5 1.95 mm to (147.8, 67.1)
- moved C4 1.88 mm to (134.6, 82.3)
- moved R5 1.86 mm to (138.4, 82.3)
- moved C3 1.78 mm to (118.1, 82.3)
- moved C1 1.69 mm to (125.2, 74.9)
- moved C2 1.69 mm to (137.9, 74.9)
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Connections:
- net Net-(J1-Pad1) renamed /~A
- net Net-(J1-Pad2) renamed /A
- net Net-(J1-Pad3) renamed /B
- net Net-(J1-Pad4) renamed /~B
- RV1 pad 3: +3V3 -> Net-(R6-Pad2)
- RV2 pad 3: +3V3 -> Net-(R6-Pad2)
- U3 pad 10: Net-(U3-Pad10) -> Net-(SW3-Pad4)
- U3 pad 21: (no net) -> Net-(U3-Pad21)
- U3 pad 3: LED1 -> LED3
- U3 pad 5: LED3 -> LED1
- U3 pad 9: Net-(SW3-Pad4) -> (no net)
- U4 pad 5: Net-(U3-Pad10) -> Net-(U3-Pad21)
Routing:
- net GNDD: track 0.00 -> 218.0 mm, vias 0 -> 10
- net +3V3: track 0.00 -> 111.7 mm, vias 0 -> 1
- net Net-(U3-Pad11): track 0.00 -> 71.5 mm, vias 0 -> 1
- net Net-(U3-Pad12): track 0.00 -> 64.2 mm
- net Net-(U3-Pad13): track 0.00 -> 53.1 mm, vias 0 -> 1
- net Net-(U3-Pad21): track 0.00 -> 36.0 mm, vias 0 -> 1
- net Net-(U3-Pad20): track 0.00 -> 28.9 mm, vias 0 -> 1
- net Net-(R6-Pad2): track 0.00 -> 23.3 mm
- net LED1: track 0.00 -> 22.0 mm
- net Net-(J2-Pad3): track 0.00 -> 19.5 mm
- net Net-(SW3-Pad4): track 0.00 -> 19.0 mm
- net /~A: track 0.00 -> 16.3 mm
- net /~B: track 0.00 -> 16.0 mm
- net LED2: track 0.00 -> 15.7 mm
- net Net-(SW3-Pad3): track 0.00 -> 14.8 mm
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Other:
- outline, holes or cut-outs redrawn
- net class Default: clearance 0.2032 -> 0.1524; trace_width 0.2032 -> 0.1524; via_dia 0.8 -> 0.762; via_drill 0.4 -> 0.381
- rule pad_to_mask_clearance: 0.051 -> 0.0508
- rule solder_mask_min_width: 0.25 -> 0.1016
- rule trace_clearance: 0.2032 -> 0.1524
- rule via_min_drill: 0.3 -> 0.254
- rule via_min_size: 0.4 -> 0.508
- board text added: "1"
- board text added: "14"
- board text added: "20"
- board text added: "33"
- board text added: "Stepper Motor Analyzer - Reference Design Rev 1.0, Open Source Hardware"

Commit message: Work in progress
Parts:
- C3, C4: value 0.1uF -> 0.22uF
- moved C5 3.57 mm to (148.3, 70.6)
Connections:
- C1 pad 2: +3V3 -> +3V3A
- C2 pad 2: +3V3 -> +3V3A
- C5 pad 1: +3V3 -> +3V3D
- R6 pad 1: +3V3 -> +3V3A
- U1 pad 10: +3V3 -> +3V3A
- U2 pad 10: +3V3 -> +3V3A
- U3 pad 16: +3V3 -> +3V3D
- U3 pad 22: (no net) -> Net-(SW2-Pad2)
- U3 pad 23: (no net) -> Net-(SW1-Pad2)
- U3 pad 25: Net-(SW2-Pad2) -> (no net)
- U3 pad 26: Net-(SW1-Pad2) -> (no net)
- U3 pad 31: +3V3 -> +3V3A
- U4 pad 2: +3V3 -> +3V3D
Routing:
- net +3V3: track 111.7 -> 0.00 mm, vias 1 -> 0
- net +3V3A: track 0.00 -> 72.7 mm, vias 0 -> 1
- net Net-(SW2-Pad2): track 6.50 -> 63.6 mm, vias 0 -> 2
- net +3V3D: track 0.00 -> 45.5 mm
- net POT1: track 0.00 -> 44.1 mm
- net POT2: track 0.00 -> 43.2 mm
- net Net-(SW1-Pad2): track 6.50 -> 48.3 mm, vias 0 -> 2
- net GNDD: track 218.0 -> 244.8 mm
- net Net-(U3-Pad11): track 71.5 -> 65.8 mm
- net Net-(U3-Pad21): track 36.0 -> 38.7 mm
- net Net-(U3-Pad13): track 53.1 -> 55.5 mm
- net Net-(U3-Pad12): track 64.2 -> 62.4 mm
- net Net-(J2-Pad2): track 7.80 -> 6.07 mm, vias 1 -> 0
- net Net-(SW3-Pad4): track 19.0 -> 17.5 mm
- net Net-(SW3-Pad3): track 14.8 -> 13.5 mm
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Other:
- board text added: "CUTOUT"

Commit message: Generated gerbers
Routing:
- net +3V3D: track 45.5 -> 44.7 mm
- added copper zone on B.Cu, net GNDD

Commit message: Work in progress.
Parts:
- removed C5: 0.1uF, stepper_analyzer:C_0603_1608Metric
- removed R6: 400R, stepper_analyzer:R_0603_1608Metric
- removed RV1, RV2: 10K, stepper_analyzer:Potentiometer_TT_P0915N
- removed SW1, SW2: SW_Push, stepper_analyzer:SW_PUSH_6mm_H7.3mm
- removed SW3: SW_DIP_x04, stepper_analyzer:SW_DIP_SPSTx04_Slide_Copal_CHS-04B_W7.62mm_P1.27mm
- removed U4: TFT, stepper_analyzer:DIP-TFT
- added J3: Conn_01x05, Connector_Molex:Molex_KK-254_AE-6410-05A_1x05_P2.54mm_Vertical, F.Cu at (144.3, 106.9)
- added J4: Conn_01x04_Female, Connector_PinHeader_2.54mm:PinHeader_1x04_P2.54mm_Vertical, F.Cu at (151.6, 79.5)
- C1, C2: value 0.1uF -> C_Small
- C3, C4: value 0.22uF -> C_Small
- R1, R2, R3: value 3K -> R_Small_US
- R4, R5: value 330R -> R_Small_US
- U1, U2: value ACS70331EESATR-2P5U3 -> ACS70331
- U3: value Teensy 4,0 -> Teensy4-stepper_analyzer
- moved H4 42.7 mm to (149.9, 106.7)
- moved H3 39.4 mm to (149.9, 64.8)
- moved H2 16.5 mm to (115.6, 106.7)
- moved TP3 15.5 mm to (129.8, 107.4)
- moved R3 13.2 mm to (131.3, 104.2), turned to 90 degrees
- moved D1 12.5 mm to (121.2, 104.2), turned to 270 degrees
- moved D3 11.9 mm to (129.8, 104.2), turned to 270 degrees
- moved TP2 11.8 mm to (125.5, 107.4)
- moved TP1 11.2 mm to (121.2, 107.4)
- moved R1 11.2 mm to (122.7, 104.1), turned to 90 degrees
- moved R2 10.2 mm to (127.0, 104.2), turned to 90 degrees
- moved D2 10.2 mm to (125.5, 104.2), turned to 270 degrees
- moved C3 0.51 mm to (117.6, 82.3)
- moved R4 0.51 mm to (121.4, 82.3)
- moved C4 0.25 mm to (134.9, 82.3)
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- renumbered H4 to H2, H2 to H3, H3 to H4, CH1 to TP4, GND1 to TP5, CH2 to TP6
Connections:
- JP1 pad 3: POT1 -> /POT1
- JP2 pad 3: POT2 -> /POT2
- U3 pad 10: Net-(SW3-Pad4) -> (no net)
- U3 pad 11: Net-(U3-Pad11) -> (no net)
- U3 pad 12: Net-(U3-Pad12) -> (no net)
- U3 pad 13: Net-(U3-Pad13) -> (no net)
- U3 pad 16: +3V3D -> (no net)
- U3 pad 20: Net-(U3-Pad20) -> (no net)
- U3 pad 21: Net-(U3-Pad21) -> /SERIAL_OUT
- U3 pad 22: Net-(SW2-Pad2) -> /SERIAL_IN
- U3 pad 23: Net-(SW1-Pad2) -> (no net)
- U3 pad 33: (no net) -> /+5V
- U3 pad 6: Net-(SW3-Pad1) -> (no net)
- U3 pad 7: Net-(SW3-Pad2) -> (no net)
- U3 pad 8: Net-(SW3-Pad3) -> (no net)
Routing:
- net GNDD: track 244.8 -> 154.2 mm, vias 10 -> 7
- net /+5V: track 0.00 -> 66.8 mm
- net Net-(U3-Pad11): track 65.8 -> 0.00 mm, vias 1 -> 0
- net Net-(SW2-Pad2): track 63.6 -> 0.00 mm, vias 2 -> 0
- net Net-(U3-Pad12): track 62.4 -> 0.00 mm
- net Net-(U3-Pad13): track 55.5 -> 0.00 mm, vias 1 -> 0
- net Net-(SW1-Pad2): track 48.3 -> 0.00 mm, vias 2 -> 0
- net +3V3D: track 44.7 -> 0.00 mm
- net POT1: track 44.1 -> 0.00 mm
- net POT2: track 43.2 -> 0.00 mm
- net /SERIAL_IN: track 0.00 -> 41.6 mm
- net Net-(U3-Pad21): track 38.7 -> 0.00 mm, vias 1 -> 0
- net /SERIAL_OUT: track 0.00 -> 37.3 mm
- net Net-(U3-Pad20): track 28.9 -> 0.00 mm, vias 1 -> 0
- net /POT1: track 0.00 -> 24.4 mm
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- removed copper zone on B.Cu, net GNDD
Other:
- board size 81.3 x 66 mm -> 41.9 x 49.5 mm
- board text added: "0V"
- board text added: "5V"
- board text added: "RX"
- board text added: "Stepper Analyzer Rev 1.1, OSH"
- board text added: "TX"
- board text removed: "14"
- board text removed: "CUTOUT"
- board text removed: "Stepper Motor Analyzer - Reference Design Rev 1.0, Open Source Hardware"

Commit message: Generated gerbers.
Parts:
- C1, C2, C3, C4: value C_Small -> 100nf
- J3: footprint Connector_Molex:Molex_KK-254_AE-6410-05A_1x05_P2.54mm_Vertical -> stepper_analyzer:Molex_KK-254_AE-6410-05A_1x05_P2.54mm_Vertical
- R1, R2, R3: value R_Small_US -> 3K3
- R4, R5: value R_Small_US -> 330R
Routing:
- net /SERIAL_OUT: track 37.3 -> 40.0 mm
- net LED2: track 15.9 -> 13.6 mm
- net GNDD: track 154.2 -> 156.3 mm
- net LED1: track 8.06 -> 8.82 mm, vias 0 -> 2
- added copper zone on B.Cu, net GNDD
Other:
- outline, holes or cut-outs redrawn
- board text added: "CH1"
- board text added: "GND"
- board text added: "Nextion 3.5"
- board text added: "Not Used"
- board text added: "Stepper Analyzer Rev 1.1, OSH Use with Nextion 3.5""
- board text added: "Teensy 4.0"
- board text removed: "Stepper Analyzer Rev 1.1, OSH"

Commit message: Version 1.1
Parts:
- J4: footprint Connector_PinHeader_2.54mm:PinHeader_1x04_P2.54mm_Vertical -> stepper_analyzer:PinHeader_1x04_P2.54mm_Vertical
- U1, U2: footprint Sensor_Current:Allegro_QFN-12-10-1EP_3x3mm_P0.5mm -> stepper_analyzer:Allegro_QFN-12-10-1EP_3x3mm_P0.5mm
Routing:
- net GNDD: track 156.3 -> 135.1 mm
- net Net-(JP1-Pad1): track 5.66 -> 6.63 mm
