File: pulser/kicad/pulser.kicad_pcb (KiCad board)
At the start: 2 copper layers, 90 x 70 mm, 47 parts, among them J1 Screw_Terminal_01x02, J2 Screw_Terminal_01x02, J3 Conn_01x06_Male, J4 Screw_Terminal_01x02, J5 Conn_01x07_Male, Q1 DMN1019UVT-7, Q2 DMN1019UVT-7, SW1 SW_Push, SW2 SW_Push, SW3 SW_Push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

Commit message: Narrower fuse slot. Also regenerated gerbers.
Parts:
- D1: value S10ML-TP -> SB2060TA
- D3, D5: value Z3SMCxxx -> MBRX120LF-TP
- F1: footprint Fuse:Fuse_Blade_Mini_directSolder -> pulsar:Fuse_Blade_Mini_directSolder
