File: stlink_adapter/stlink_adapter.kicad_pcb (KiCad board)
At the start: 2 copper layers, 21.6 x 30.5 mm, 5 parts, among them J1 Conn_02x10_Odd_Even, J2 Conn_01x03_Male, J3 Conn_01x04_Female

Commit message: Tweaked and generated gerbers.
Parts:
- J2: value Conn_01x03_Male -> Conn_01x02_Male; footprint Connector_PinHeader_2.54mm:PinHeader_1x03_P2.54mm_Vertical -> Connector_PinHeader_2.54mm:PinHeader_1x02_P2.54mm_Vertical
- moved J2 5.08 mm to (128.3, 85.1), turned to 270 degrees
- moved D1 0.80 mm to (130.7, 80.4)
- moved R1 0.80 mm to (128.0, 80.4)
Connections:
- J2 pad 1: Net-(J1-Pad1) -> Net-(J1-Pad19)
- J2 pad 2: Net-(J2-Pad2) -> Net-(J1-Pad1)
- J3 pad 4: Net-(J2-Pad2) -> Net-(J1-Pad1)
- R1 pad 1: Net-(J2-Pad2) -> Net-(J1-Pad1)
Routing:
- net Net-(J2-Pad2): track 24.9 -> 0.00 mm
- net Net-(D1-Pad1): track 38.0 -> 38.8 mm
- net Net-(J1-Pad1): track 34.6 -> 35.4 mm
Other:
- board text removed: "INT"

Commit message: Flushing pending changes in misc/...
Parts:
- moved D1 15.5 mm to (129.5, 64.9)
- moved R1 15.5 mm to (126.9, 64.9)
- moved J2 6.48 mm to (121.9, 86.4), turned to 180 degrees
- moved J3 6.35 mm to (121.9, 78.7)
Routing:
- net Net-(J1-Pad19): track 18.0 -> 10.0 mm
- net Net-(D1-Pad1): track 38.8 -> 42.9 mm
- net Net-(J1-Pad1): track 35.4 -> 38.1 mm
- net Net-(J1-Pad7): track 9.20 -> 8.67 mm
- net Net-(J1-Pad9): track 9.20 -> 8.67 mm
Other:
- board text added: "EXT 3.3V"
- board text added: "STLINK/V2 SWD ADAPTER"
- board text removed: "3.3V"
- board text removed: "EXT"
- board text removed: "STLINK-V2 SWD ADAPTER"

Commit message: Cleaned up the design.
Parts:
- D1: footprint LED_SMD:LED_0603_1608Metric_Pad1.05x0.95mm_HandSolder -> stlink_adapter:LED_0603_1608Metric_Pad1.05x0.95mm_HandSolder
- J1: footprint Connector_PinHeader_2.54mm:PinHeader_2x10_P2.54mm_Vertical -> stlink_adapter:PinHeader_2x10_P2.54mm_Vertical
- J2: footprint Connector_PinHeader_2.54mm:PinHeader_1x02_P2.54mm_Vertical -> stlink_adapter:PinHeader_1x02_P2.54mm_Vertical
- J3: footprint Connector_PinHeader_2.54mm:PinHeader_1x04_P2.54mm_Vertical -> stlink_adapter:PinHeader_1x04_P2.54mm_Vertical
- R1: footprint Resistor_SMD:R_0603_1608Metric_Pad1.05x0.95mm_HandSolder -> stlink_adapter:R_0603_1608Metric_Pad1.05x0.95mm_HandSolder
Connections:
- J1 pad 10: (no net) -> unconnected-(J1-Pin_10-Pad10)
- J1 pad 11: (no net) -> unconnected-(J1-Pin_11-Pad11)
- J1 pad 12: (no net) -> unconnected-(J1-Pin_12-Pad12)
- J1 pad 13: (no net) -> unconnected-(J1-Pin_13-Pad13)
- J1 pad 14: (no net) -> unconnected-(J1-Pin_14-Pad14)
- J1 pad 15: (no net) -> unconnected-(J1-Pin_15-Pad15)
- J1 pad 16: (no net) -> unconnected-(J1-Pin_16-Pad16)
- J1 pad 17: (no net) -> unconnected-(J1-Pin_17-Pad17)
- J1 pad 18: (no net) -> unconnected-(J1-Pin_18-Pad18)
- J1 pad 2: (no net) -> unconnected-(J1-Pin_2-Pad2)
- J1 pad 20: (no net) -> unconnected-(J1-Pin_20-Pad20)
- J1 pad 3: (no net) -> unconnected-(J1-Pin_3-Pad3)
- J1 pad 5: (no net) -> unconnected-(J1-Pin_5-Pad5)
Other:
- net class Default removed
