File: pulser2/kicad/pulser.kicad_pcb (KiCad board)
At the start: 2 copper layers, 90 x 70 mm, 44 parts, among them J1 Screw_Terminal_01x02, J2 Screw_Terminal_01x02, J4 Screw_Terminal_01x02, J5 Conn_01x07_Male, Q1 DMN1019UVT-7, Q2 DMN1019UVT-7, SW1 SW_Push, SW2 SW_Push, SW3 SW_Push, SW4 SW_Coded_SH-7010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

Commit message: Final verstion. Ordered as V1.1.
Parts:
- moved C4 1.52 mm to (126.8, 99.7)
- moved U3 1.52 mm to (126.6, 94.5)
- moved TP4 0.23 mm to (100.3, 104.3)
- moved R1 0.13 mm to (138.7, 126.4)
- turned R11 to 0 degrees
Routing:
- net Net-(J4-Pad2): track 24.0 -> 20.2 mm
- net /GATE: track 48.7 -> 51.3 mm
- net /+24V: track 99.1 -> 101.4 mm
- net +5V: track 154.9 -> 156.7 mm
- net Net-(R10-Pad2): track 11.7 -> 12.8 mm
