File: duet3d_accel/rrf_accel.kicad_sch (KiCad schematic)
At the start: 13 parts, among them J1 Conn_02x05_Odd_Even, U1 LIS3DH

Commit message: Tweaked the layout
Parts:
- J1: JLCRotOffset (none) -> 90
Other:
- note removed: "TODO: Add via holes to the connector pads"
- note removed: "TODO: Make the IC footprint manual solder friendly"
Changed lines of the file:
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@@
     (stroke (width 0) (type default))
-  )
-  (text "TODO: Add via holes to the connector pads" (at 29.845 32.385 0)
-    (effects (font (size 2.54 2.54) (thickness 0.508) bold (color 255 0 0 1)) (justify left bottom))
-  )
-  (text "TODO: Make the IC footprint manual solder friendly"
-    (at 30.48 60.325 0)
-    (effects (font (size 2.54 2.54) (thickness 0.508) bold (color 255 0 0 1)) (justify left bottom))
   )
   (text "TODO: Verify footprint" (at 29.845 47.625 0)
@@
       (effects (font (size 1.27 1.27)) hide)
     )
+    (property "JLCRotOffset" "90" (at 69.85 101.6 0)
+      (effects (font (size 1.27 1.27)) hide)
+    )
