File: duet3d_accel/rrf_accel.kicad_sch (KiCad schematic)
At the start: 13 parts, among them J1 Conn_02x05_Odd_Even, U1 LIS3DH

Commit message: First layout.
Parts:
- C1: value C_Small -> 10uf; footprint (none) -> Capacitor_SMD:C_0603_1608Metric_Pad1.08x0.95mm_HandSolder; LCSC (none) -> C96446
- C2: value C_Small -> 100n; footprint (none) -> Capacitor_SMD:C_0402_1005Metric_Pad0.74x0.62mm_HandSolder; LCSC (none) -> C96446
- C3, C4: value C_Small -> 470pf; footprint (none) -> Capacitor_SMD:C_0603_1608Metric_Pad1.08x0.95mm_HandSolder; LCSC (none) -> C1620
- D1: footprint (none) -> LED_SMD:LED_0603_1608Metric_Pad1.05x0.95mm_HandSolder; LCSC (none) -> C72043
- J1: footprint (none) -> duet3d_accel:PinHeader_2x05_P2.54mm_Vertical_SMD; LCSC (none) -> C236047
- R1, R2, R4, R5, R6: value R_US -> 62R; footprint (none) -> Resistor_SMD:R_0402_1005Metric_Pad0.72x0.64mm_HandSolder; LCSC (none) -> C25120
- R3: value R_US -> 220R; footprint (none) -> Resistor_SMD:R_0402_1005Metric_Pad0.72x0.64mm_HandSolder; LCSC (none) -> C25091
- U1: LCSC (none) -> C15134
Connections:
- net CS: now also J1.1 (Pin_1)
- net INT: now also J1.3 (Pin_3)
- net MISO: now also J1.6 (Pin_6)
- net MOSI: now also J1.5 (Pin_5)
- net SCK: now also J1.4 (Pin_4)
Other:
- note added: "TODO: Add via holes to the connector pads"
- note added: "TODO: Make the IC footprint manual solder friendly"
- note added: "TODO: Verify footprint"
- moved on the sheet: C1, C2, C3, C4, J1, R1, R2, R4, R5, R6, U1

Commit message: Updated schematic.
Parts:
- J1: LCSC C236047 -> C383605
Changed lines of the file:
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@@
       (effects (font (size 1.27 1.27)) hide)
     )
-    (property "LCSC" "C236047" (at 69.85 101.6 0)
+    (property "LCSC" "C383605" (at 69.85 101.6 0)
       (effects (font (size 1.27 1.27)) hide)
     )
